Commit message: initialize to sim working mode

File: src/st_arm_description/urdf/st_arm.urdf (robot description, URDF)
Before this commit: robot st_arm, 9 links, 8 joints
Links:
- link base_link: mass 0.594687468826075 -> 0.068254; geometry collision mesh filename=package://st_arm_description/meshes/stl/base_link.STL; visual mesh filename=package://st_arm_description/meshes/stl/base_link.STL
- link elbow_pitch_link: mass 0.170291975194639 -> 0.15458; geometry collision mesh filename=package://st_arm_description/meshes/stl/elbow_pitch_link.STL; visual mesh filename=package://st_arm_description/meshes/stl/elbow_pitch_link.STL
- link gripper_left_link: mass 0.0001 -> 0.0151655067348166
- link gripper_right_link: mass 0.0001 -> 0.0151655067348167
- link shoulder_pitch_link: mass 0.653267805710522 -> 0.24697; geometry collision mesh filename=package://st_arm_description/meshes/stl/shoulder_pitch_link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; visual mesh filename=package://st_arm_description/meshes/stl/shoulder_pitch_link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
- link shoulder_yaw_link: mass 0.552307334689627 -> 0.11951; geometry collision mesh filename=package://st_arm_description/meshes/stl/shoulder_yaw_link.S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; visual mesh filename=package://st_arm_description/meshes/stl/shoulder_yaw_link.S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
- link wrist_pitch_link: mass 0.0923460959053665 -> 0.04488; geometry collision mesh filename=package://st_arm_description/meshes/stl/wrist_pitch_link.STL; visual mesh filename=package://st_arm_description/meshes/stl/wrist_pitch_link.STL
- link wrist_roll_link: mass 0.0869629421685106 -> 0.04488; geometry collision mesh filename=package://st_arm_description/meshes/stl/wrist_roll_link.STL; visual mesh filename=package://st_arm_description/meshes/stl/wrist_roll_link.STL
- link wrist_yaw_link: mass 0.148763165360562 -> 0.0830727105278852; geometry collision mesh filename=package://st_arm_description/meshes/stl/wrist_yaw_link.STL; visual mesh filename=package://st_arm_description/meshes/stl/wrist_yaw_link.STL
Joints:
- joint elbow_pitch_joint: limit lower=-2.9 upper=2.9 effort=1 velocity=1 -> lower=-0.1 upper=2.8 effort=1 velocity=1
- joint gripper_left_joint: limit lower=-0.03 upper=0 effort=1 velocity=1 -> lower=-0.05 upper=0 effort=1 velocity=1; origin xyz=0.083595 0 0 rpy=0 0 0 -> xyz=0.083595 0.0016804 0 rpy=0 0 0
- joint gripper_right_joint: limit lower=-0.03 upper=0 effort=1 velocity=1 -> lower=-0.05 upper=0 effort=1 velocity=1; origin xyz=0.083595 0 0 rpy=0 0 0 -> xyz=0.083595 0.0016804 0 rpy=0 0 0
- joint shoulder_pitch_joint: limit lower=-3.9 upper=0.76 effort=1 velocity=1 -> lower=-3.14 upper=0.1 effort=1 velocity=1; origin xyz=0 0 0.1019 rpy=0 0 0 -> xyz=0 0 0.1024 rpy=0 0 0
- joint wrist_pitch_joint: limit lower=-1.57 upper=1.57 effort=1 velocity=1 -> lower=-2.8 upper=3.5 effort=1 velocity=1
- joint wrist_roll_joint: limit lower=-1.57 upper=1.57 effort=1 velocity=1 -> lower=-3.14 upper=3.14 effort=1 velocity=1
